Commit message: Partie 2 : choix de la personne, couleur des vetements, re-identification, camera en haut
- Couleur des vetements par ID (clothing_color, vote sur 15 images), champ Track.color
- Fenetre target_chooser : clic sur une personne -> /target/select ; selection manuelle
- Pulls rouge / vert / violet pour les 3 personnes, monde agrandi a 18 x 14 m
- Distance par la hauteur de la silhouette au-dela de la portee du LiDAR
- Re-identification par la couleur, garde contre le vol d'ID, doublons de la cible
- ByteTrack : track_buffer 90 (bytetrack_person.yaml)
- Camera en haut du robot (26 cm, mat), SDF et URDF
- Rosbags : /tracks et /target/select ; README et rapport mis a jour (videos de demo)

File: tb_bringup/urdf/tb3_burger_cam.urdf (robot description, URDF)
Before this commit: robot turtlebot3_burger_cam, 10 links, 9 joints
Joints:
- joint camera_joint: origin xyz=0.040 -0.000 0.110 rpy=0 0 0 -> xyz=-0.035 0.000 0.241 rpy=0 0 0
